Commit message: Organize ping pong arm RL experiments

File: urdf/braccioLight/braccioLight.urdf (robot description, URDF)
Before this commit: robot umirobot_l1, 5 links, 4 joints
Links:
- link end_effector: geometry collision mesh filename=file://endEffector.stl scale=0.5 0.5 0.5; visual mesh filename=file://endEffector.stl scale=0.5 0.5 0.5
- link robot_base: geometry collision mesh filename=file://piece1.stl scale=0.01 0.01 0.01; visual mesh filename=file://piece1.stl scale=0.01 0.01 0.01
- link umirobot_l2_cover: geometry collision mesh filename=file://piece2.stl scale=0.01 0.01 0.01; visual mesh filename=file://piece2.stl scale=0.01 0.01 0.01
- link umirobot_l3: geometry collision mesh filename=file://piece3.stl scale=0.01 0.01 0.01; visual mesh filename=file://piece3.stl scale=0.01 0.01 0.01
- link umirobot_l4: geometry collision mesh filename=file://piece4.stl scale=0.01 0.01 0.01; visual mesh filename=file://piece4.stl scale=0.01 0.01 0.01

File: urdf/paddle/braccioConRacket.urdf (robot description, URDF)
Before this commit: robot umirobot_l1, 5 links, 4 joints
Links:
- link Racket: geometry visual mesh filename=file://braccioConRacket_Racket_vis_1.dae
- link robot_base: geometry collision mesh filename=file://braccioConRacket_robot_base_coll_1.dae; visual mesh filename=file://braccioConRacket_robot_base_vis_1.dae
- link umirobot_l2_cover: geometry collision mesh filename=file://braccioConRacket_umirobot_l2_cover_coll_1.dae; visual mesh filename=file://braccioConRacket_umirobot_l2_cover_vis_1.dae
- link umirobot_l3: geometry collision mesh filename=file://braccioConRacket_umirobot_l3_coll_1.dae; visual mesh filename=file://braccioConRacket_umirobot_l3_vis_1.dae
- link umirobot_l4: geometry collision mesh filename=file://braccioConRacket_umirobot_l4_coll_1.dae; visual mesh filename=file://braccioConRacket_umirobot_l4_vis_1.dae

File: urdf/paddle/racket.urdf (robot description, URDF)
Before this commit: robot ping_pong_racket, 1 links, 0 joints
Links:
- link racket: geometry collision mesh filename=Racket.stl scale=0.001 0.001 0.001; visual mesh filename=Racket.stl scale=0.001 0.001 0.001

File: urdf/table/table.urdf (robot description, URDF)
Before this commit: robot ping_pong_table, 1 links, 0 joints
Links:
- link table: geometry collision box size=2.8 1.6 0.05; visual mesh filename=../table/tavoloGirato.stl scale=0.01 0.01 0.01
